File: hardware/MegadriveControllerToUSB.sch (KiCad schematic (older format))
At the start: 13 parts, among them CON1 AVR-ISP6, J1 USB, J2 DB9, U1 ATMEGA32U2-AU, X1 16Mhz

Commit message: Set pin numbers properly. Need to test again. Removing some kicad temp files.
Connections:
- net labels added: DATA0_PIN, DATA1_PIN, DATA2_PIN, DATA3_PIN, DATA4_PIN, DATA5_PIN
- net labels removed: B_A_BUTTON, C_START_BUTTON, DOWN_Y, LEFT_X, RIGHT_MODE, UP_Z
Changed lines of the file:
@@
 Sheet 1 1
 Title ""
-Date "4 aug 2014"
+Date "16 nov 2014"
 Rev ""
 Comp ""
@@
 SELECT_CLK
 Text GLabel 8700 1400 0    60   Input ~ 0
-B_A_BUTTON
+DATA5_PIN
 Text GLabel 9450 1500 0    60   Input ~ 0
-RIGHT_MODE
+DATA3_PIN
 Text GLabel 9450 1900 0    60   Input ~ 0
-DOWN_Y
+DATA1_PIN
 $Comp
 L VCC #PWR010
@@
 	9600 1300 9700 1300
 Text GLabel 8700 2000 0    60   Input ~ 0
-C_START_BUTTON
+DATA4_PIN
 Text GLabel 9450 1700 0    60   Input ~ 0
-LEFT_X
+DATA2_PIN
 Text GLabel 9450 2100 0    60   Input ~ 0
-UP_Z
+DATA0_PIN
 Text GLabel 4250 4800 0    60   Input ~ 0
 RESET
@@
 	9450 2100 9700 2100
 Text GLabel 7000 4800 2    60   Input ~ 0
-B_A_BUTTON
+DATA5_PIN
 Text GLabel 7700 4900 2    60   Input ~ 0
-RIGHT_MODE
+DATA3_PIN
 Text GLabel 7000 5000 2    60   Input ~ 0
-LEFT_X
+DATA2_PIN
 Text GLabel 7700 5100 2    60   Input ~ 0
 SELECT_CLK
 Text GLabel 7000 5200 2    60   Input ~ 0
-DOWN_Y
+DATA1_PIN
 Text GLabel 7700 5300 2    60   Input ~ 0
-C_START_BUTTON
+DATA4_PIN
 Text GLabel 7000 5400 2    60   Input ~ 0
-UP_Z
+DATA0_PIN
 Wire Wire Line
 	6700 4800 7000 4800
